File: electrical/PID Motor DC_Schematic/pid motor DC.sch (EAGLE design)
At the start: 6 parts

Commit message: rev pin name
Connections:
- net A-IA renamed MTR_CW
- net A-IB renamed MTR_CCW
- net BTN_INPUT renamed BT1
- net HALL_SIGA renamed ENC_A
- net HALL_SIGB renamed ENC_B
- net POT_INPUT renamed POT
Changed lines of the file:
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@@
 <setting verticaltext="up"/>
 </settings>
-<grid distance="0.1" unitdist="inch" unit="inch" style="lines" multiple="1" display="yes" altdistance="0.01" altunitdist="inch" altunit="inch"/>
+<grid distance="0.1" unitdist="inch" unit="inch" style="lines" multiple="1" display="no" altdistance="0.01" altunitdist="inch" altunit="inch"/>
 <layers>
 <layer number="1" name="Top" color="4" fill="1" visible="no" active="no"/>
@@
 </plain>
 <moduleinsts>
-<moduleinst name="HG7661_MOTOR_DRIVER" module="HG7661" x="203.2" y="76.2" rot="R270" grouprefs="DC_MOTOR_MODULE">
-<attribute name="NAME" value="HG7661_MOTOR_DRIVER" x="204.216" y="91.948" size="2.032" layer="95" align="bottom-center"/>
+<moduleinst name="HG7881_MOTOR_DRIVER" module="HG7661" x="203.2" y="76.2" rot="R270" grouprefs="DC_MOTOR_MODULE">
+<attribute name="NAME" value="HG7881_MOTOR_DRIVER" x="204.216" y="91.948" size="2.032" layer="95" align="bottom-center"/>
 </moduleinst>
-<moduleinst name="12V_PSU" module="12V_PSU" x="119.38" y="38.1" grouprefs="SUPPLY_MODULE">
-<attribute name="NAME" value="12V_PSU" x="119.38" y="38.1" size="2.032" layer="95" align="bottom-center"/>
+<moduleinst name="12V_PSU" module="12V_PSU" x="116.84" y="38.608" grouprefs="SUPPLY_MODULE">
+<attribute name="NAME" value="12V_PSU" x="116.84" y="38.608" size="2.032" layer="95" align="bottom-center"/>
 </moduleinst>
 </moduleinsts>
@@
 <attribute name="VALUE" x="79.375" y="88.265" size="1.778" layer="96"/>
 </instance>
-<instance part="SUPPLY3" gate="GND" x="149.86" y="38.1" smashed="yes" grouprefs="SUPPLY_MODULE">
-<attribute name="VALUE" x="147.955" y="34.925" size="1.778" layer="96"/>
-</instance>
-<instance part="P+3" gate="1" x="149.86" y="50.8" smashed="yes" grouprefs="SUPPLY_MODULE">
-<attribute name="VALUE" x="147.32" y="45.72" size="1.778" layer="96" rot="R90"/>
+<instance part="SUPPLY3" gate="GND" x="147.32" y="38.608" smashed="yes" grouprefs="SUPPLY_MODULE">
+<attribute name="VALUE" x="145.415" y="35.433" size="1.778" layer="96"/>
+</instance>
+<instance part="P+3" gate="1" x="147.32" y="51.308" smashed="yes" grouprefs="SUPPLY_MODULE">
+<attribute name="VALUE" x="144.78" y="46.228" size="1.778" layer="96" rot="R90"/>
 </instance>
 <instance part="P+4" gate="1" x="78.74" y="78.74" smashed="yes" grouprefs="HMI_MODULE">
@@
 <segment>
 <pinref part="SUPPLY7" gate="GND" pin="GND"/>
-<portref moduleinst="HG7661_MOTOR_DRIVER" port="GND"/>
+<portref moduleinst="HG7881_MOTOR_DRIVER" port="GND"/>
 <wire x1="200.66" y1="55.88" x2="200.66" y2="53.34" width="0.1524" layer="91" grouprefs="DC_MOTOR_MODULE"/>
 </segment>
 <segment>
 <portref moduleinst="12V_PSU" port="12V-"/>
-<wire x1="139.7" y1="43.18" x2="148.844" y2="43.18" width="0.1524" layer="91" grouprefs="SUPPLY_MODULE"/>
-<wire x1="148.844" y1="43.18" x2="149.86" y2="42.164" width="0.1524" layer="91" grouprefs="SUPPLY_MODULE"/>
+<wire x1="137.16" y1="43.688" x2="146.304" y2="43.688" width="0.1524" layer="91" grouprefs="SUPPLY_MODULE"/>
+<wire x1="146.304" y1="43.688" x2="147.32" y2="42.672" width="0.1524" layer="91" grouprefs="SUPPLY_MODULE"/>
 <pinref part="SUPPLY3" gate="GND" pin="GND"/>
-<wire x1="149.86" y1="42.164" x2="149.86" y2="40.64" width="0.1524" layer="91" grouprefs="SUPPLY_MODULE"/>
+<wire x1="147.32" y1="42.672" x2="147.32" y2="41.148" width="0.1524" layer="91" grouprefs="SUPPLY_MODULE"/>
 </segment>
 </net>
@@
 <segment>
 <pinref part="P+7" gate="1" pin="+12V"/>
-<portref moduleinst="HG7661_MOTOR_DRIVER" port="VS"/>
+<portref moduleinst="HG7881_MOTOR_DRIVER" port="VS"/>
 <wire x1="205.74" y1="55.88" x2="205.74" y2="53.34" width="0.1524" layer="91" grouprefs="DC_MOTOR_MODULE"/>
 </segment>
@@
 <segment>
 <portref moduleinst="12V_PSU" port="12V+"/>
-<wire x1="139.7" y1="45.72" x2="148.59" y2="45.72" width="0.1524" layer="91" grouprefs="SUPPLY_MODULE"/>
-<wire x1="148.59" y1="45.72" x2="149.86" y2="46.99" width="0.1524" layer="91" grouprefs="SUPPLY_MODULE"/>
+<wire x1="137.16" y1="46.228" x2="146.05" y2="46.228" width="0.1524" layer="91" grouprefs="SUPPLY_MODULE"/>
+<wire x1="146.05" y1="46.228" x2="147.32" y2="47.498" width="0.1524" layer="91" grouprefs="SUPPLY_MODULE"/>
 <pinref part="P+3" gate="1" pin="+12V"/>
-<wire x1="149.86" y1="46.99" x2="149.86" y2="48.26" width="0.1524" layer="91" grouprefs="SUPPLY_MODULE"/>
-</segment>
-</net>
-<net name="POT_INPUT" class="0">
+<wire x1="147.32" y1="47.498" x2="147.32" y2="48.768" width="0.1524" layer="91" grouprefs="SUPPLY_MODULE"/>
+</segment>
+</net>
+<net name="POT" class="0">
 <segment>
 <pinref part="U$2" gate="G$1" pin="A0"/>
@@
 </segment>
 </net>
-<net name="BTN_INPUT" class="0">
+<net name="BT1" class="0">
 <segment>
 <pinref part="U$2" gate="G$1" pin="D7"/>
@@
 </segment>
 </net>
-<net name="HALL_SIGA" class="0">
+<net name="ENC_A" class="0">
 <segment>
 <pinref part="U$2" gate="G$1" pin="D2"/>
@@
 </segment>
 </net>
-<net name="HALL_SIGB" class="0">
+<net name="ENC_B" class="0">
 <segment>
 <pinref part="U$2" gate="G$1" pin="D3"/>
@@
 </segment>
 </net>
-<net name="A-IA" class="0">
+<net name="MTR_CW" class="0">
 <segment>
 <pinref part="U$2" gate="G$1" pin="D5"/>
@@
 </segment>
 <segment>
-<portref moduleinst="HG7661_MOTOR_DRIVER" port="A-IA"/>
+<portref moduleinst="HG7881_MOTOR_DRIVER" port="A-IA"/>
 <wire x1="187.96" y1="86.36" x2="182.88" y2="86.36" width="0.1524" layer="91" grouprefs="DC_MOTOR_MODULE"/>
 <label x="182.88" y="86.36" size="1.4224" layer="95" rot="R180" xref="yes" grouprefs="DC_MOTOR_MODULE"/>
-</segment>
-</net>
-<net name="A-IB" class="0">
-<segment>
-<pinref part="U$2" gate="G$1" pin="D6"/>
-<wire x1="147.32" y1="101.6" x2="149.86" y2="101.6" width="0.1524" layer="91" grouprefs="MICROCONTROLLER"/>
-<label x="149.86" y="101.6" size="1.4224" layer="95" xref="yes" grouprefs="MICROCONTROLLER"/>
-</segment>
-<segment>
-<portref moduleinst="HG7661_MOTOR_DRIVER" port="A-IB"/>
-<wire x1="187.96" y1="81.28" x2="182.88" y2="81.28" width="0.1524" layer="91" grouprefs="DC_MOTOR_MODULE"/>
-<label x="182.88" y="81.28" size="1.4224" layer="95" rot="R180" xref="yes" grouprefs="DC_MOTOR_MODULE"/>
 </segment>
 </net>
@@
 </segment>
 <segment>
-<portref moduleinst="HG7661_MOTOR_DRIVER" port="M1_VS"/>
+<portref moduleinst="HG7881_MOTOR_DRIVER" port="M1_VS"/>
 <wire x1="218.44" y1="86.36" x2="223.52" y2="86.36" width="0.1524" layer="91" grouprefs="DC_MOTOR_MODULE"/>
 <label x="223.52" y="86.36" size="1.4224" layer="95" xref="yes" grouprefs="DC_MOTOR_MODULE"/>
@@
 </segment>
 <segment>
-<portref moduleinst="HG7661_MOTOR_DRIVER" port="M1_GND"/>
+<portref moduleinst="HG7881_MOTOR_DRIVER" port="M1_GND"/>
 <wire x1="218.44" y1="81.28" x2="223.52" y2="81.28" width="0.1524" layer="91" grouprefs="DC_MOTOR_MODULE"/>
 <label x="223.52" y="81.28" size="1.4224" layer="95" xref="yes" grouprefs="DC_MOTOR_MODULE"/>
@@
 <segment>
 <portref moduleinst="12V_PSU" port="L"/>
-<wire x1="139.7" y1="33.02" x2="157.48" y2="33.02" width="0.1524" layer="91" grouprefs="SUPPLY_MODULE"/>
-<label x="157.48" y="33.02" size="1.4224" layer="95" xref="yes" grouprefs="SUPPLY_MODULE"/>
+<wire x1="137.16" y1="33.528" x2="154.94" y2="33.528" width="0.1524" layer="91" grouprefs="SUPPLY_MODULE"/>
+<label x="154.94" y="33.528" size="1.4224" layer="95" xref="yes" grouprefs="SUPPLY_MODULE"/>
 </segment>
 </net>
@@
 <segment>
 <portref moduleinst="12V_PSU" port="N"/>
-<wire x1="139.7" y1="30.48" x2="157.48" y2="30.48" width="0.1524" layer="91" grouprefs="SUPPLY_MODULE"/>
-<label x="157.48" y="30.48" size="1.4224" layer="95" xref="yes" grouprefs="SUPPLY_MODULE"/>
-</segment>
-</net>
+<wire x1="137.16" y1="30.988" x2="154.94" y2="30.988" width="0.1524" layer="91" grouprefs="SUPPLY_MODULE"/>
+<label x="154.94" y="30.988" size="1.4224" layer="95" xref="yes" grouprefs="SUPPLY_MODULE"/>
+</segment>
+</net>
+<net name="MTR_CCW" class="0">
+<segment>
+<pinref part="U$2" gate="G$1" pin="D6"/>
+<wire x1="147.32" y1="101.6" x2="149.86" y2="101.6" width="0.1524" layer="91" grouprefs="MICROCONTROLLER"/>
+<label x="149.86" y="101.6" size="1.4224" layer="95" xref="yes" grouprefs="MICROCONTROLLER"/>
+</segment>
+<segment>
+<portref moduleinst="HG7881_MOTOR_DRIVER" port="A-IB"/>
+<wire x1="187.96" y1="81.28" x2="182.88" y2="81.28" width="0.1524" layer="91" grouprefs="DC_MOTOR_MODULE"/>
+<label x="182.88" y="81.28" size="1.4224" layer="95" rot="R180" xref="yes" grouprefs="DC_MOTOR_MODULE"/>
+</segment>
+</net>
